File: CARP-LITE/CARP.kicad_pcb (KiCad board)
At the start: 4 copper layers, 35 x 55 mm, 96 parts, among them J1 USB_C_Receptacle_USB2.0_14P, J2 Conn_01x10, J3 Conn_01x10, J4 U.fl, SW1 SW_Push, SW2 SW_Push, U1 W25Q128JVSIMTR (16MB), U2 W25Q32RVXHJQ (2MB), U3 LM1117IMPX-3.3, U4 RP2350_60QFN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

Commit message: .
Parts:
- removed C3, C4: 10u, Capacitor_SMD:C_0805_2012Metric
- removed C30, C34, C35, C36, C38, C39, C40, C41, C42, C50: 100n, Capacitor_SMD:C_0402_1005Metric
- removed C37: 220n, Capacitor_SMD:C_0402_1005Metric
- removed C43, C44, C45: 5.1p, Capacitor_SMD:C_0402_1005Metric
- removed C46: 56p, Capacitor_SMD:C_0402_1005Metric
- removed C47: 39p, Capacitor_SMD:C_0402_1005Metric
- removed C48: 2.2p, Capacitor_SMD:C_0402_1005Metric
- removed C49: 100p, Capacitor_SMD:C_0402_1005Metric
- removed C51: 6.2p, Capacitor_SMD:C_0402_1005Metric
- removed FB1: 1k, Inductor_SMD:L_0402_1005Metric
- removed J2, J3: Conn_01x10, Connector_PinHeader_2.54mm:PinHeader_1x10_P2.54mm_Vertical
- removed L2, L4: 27n, Inductor_SMD:L_0402_1005Metric
- removed L3, L6: 56n, Inductor_SMD:L_0402_1005Metric
- removed L5, L7: 15n, Inductor_SMD:L_0402_1005Metric
- removed L8: 43n, Inductor_SMD:L_0402_1005Metric
- removed L9: 22n, Inductor_SMD:L_0402_1005Metric
- removed R14, R15: 4.7k, Resistor_SMD:R_0402_1005Metric
- removed R16: 56k, Resistor_SMD:R_0402_1005Metric
- removed R17: 18, Resistor_SMD:R_0402_1005Metric
- removed REF**: Smolhaj_Scale_0.1, Symbol:Smolhaj_Scale_0.1
- removed Y2: TG2520SMN 40MHz, Oscillator:Oscillator_SMD_SeikoEpson_TG2520SMN-xxx-xxxxxx-4Pin_2.5x2.0mm
- added H1: MountingHole, MountingHole:MountingHole_3.2mm_M3_DIN965_Pad_TopBottom, F.Cu at (449.0, 261.0)
- added H2: MountingHole, MountingHole:MountingHole_3.2mm_M3_DIN965_Pad_TopBottom, F.Cu at (417.0, 261.0)
- added H3: MountingHole, MountingHole:MountingHole_3.2mm_M3_DIN965_Pad_TopBottom, F.Cu at (417.0, 333.0)
- added H4: MountingHole, MountingHole:MountingHole_3.2mm_M3_DIN965_Pad_TopBottom, F.Cu at (449.0, 333.0)
- added J10: PYRO_2, Connector_Molex:Molex_Nano-Fit_105313-xx02_1x02_P2.50mm_Horizontal, F.Cu at (444.4, 322.8)
- added R19: 5.1k, Resistor_SMD:R_0402_1005Metric, F.Cu at (529.9, 320.0)
- added R20: 5.1k, Resistor_SMD:R_0402_1005Metric, F.Cu at (529.9, 322.0)
- added R21: 5.1k, Resistor_SMD:R_0402_1005Metric, F.Cu at (529.9, 323.9)
- added R22: 5.1k, Resistor_SMD:R_0402_1005Metric, F.Cu at (529.9, 325.9)
- added TP1: TestPoint, TestPoint:TestPoint_Pad_D1.5mm, F.Cu at (530.2, 301.8)
- added TP2: TestPoint, TestPoint:TestPoint_Pad_D1.5mm, F.Cu at (530.2, 305.3)
- added TP3: TestPoint, TestPoint:TestPoint_Pad_D1.5mm, F.Cu at (530.2, 308.9)
- C26: value 1.5n -> 100u; footprint Capacitor_SMD:C_0402_1005Metric -> Capacitor_SMD:C_0603_1608Metric
- C28: value 4.7u -> 10u; footprint Capacitor_SMD:C_0805_2012Metric -> Capacitor_SMD:C_0603_1608Metric
- C29: value 100n -> 1u; footprint Capacitor_SMD:C_0402_1005Metric -> Capacitor_SMD:C_0603_1608Metric
- C7: footprint Capacitor_SMD:C_0805_2012Metric -> Capacitor_SMD:C_0603_1608Metric
- J4: value U.fl -> 2S XT30; footprint Connector_Coaxial:U.FL_Hirose_U.FL-R-SMT-1_Vertical -> Connector_AMASS:AMASS_XT30PW-M_1x02_P2.50mm_Horizontal
- U3: value LM1117IMPX-3.3 -> 3V3 LDO
- U7: value CC1200 -> 5V LDO; footprint Package_DFN_QFN:QFN-32-1EP_5x5mm_P0.5mm_EP3.45x3.45mm -> Package_TO_SOT_SMD:SOT-223-3_TabPin2
- moved C28 57.6 mm to (536.2, 322.7), turned to 0 degrees
- moved C27 52.8 mm to (532.7, 320.0), turned to 0 degrees
- moved C29 50.4 mm to (536.2, 325.2), turned to 0 degrees
- moved C31 47.9 mm to (532.7, 321.9), turned to 0 degrees
- moved U7 47.7 mm to (533.3, 314.9)
- moved C26 46.0 mm to (536.2, 320.2)
- moved C33 45.0 mm to (532.7, 325.9), turned to 0 degrees
- moved C32 43.9 mm to (532.7, 323.9), turned to 0 degrees
- moved C12 33.7 mm to (469.2, 309.8)
- moved C16 33.2 mm to (469.8, 311.0)
- moved C14 29.3 mm to (470.2, 315.8)
- moved J4 29.2 mm to (535.7, 344.6), turned to 0 degrees
- moved C18 21.9 mm to (469.5, 308.0)
- moved JP1 20.4 mm to (464.5, 302.1)
- moved C21 19.1 mm to (469.9, 298.2)
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Connections:
- C23 pad 1: VBUS -> +5V
- C26 pad 1: Net-(U7-LPF1) -> +5V
- C26 pad 2: Net-(U7-LPF0) -> GND
- C27 pad 1: +3.3VA -> GND
- C27 pad 2: GND -> Net-(C27-Pad2)
- C28 pad 1: +3.3VA -> +2S
- C29 pad 1: +3.3VA -> /GPIO26_ADC0
- C31 pad 1: Net-(U7-DCPL_XOSC) -> GND
- C31 pad 2: GND -> /GPIO28
- C32 pad 1: +3.3VA -> GND
- C32 pad 2: GND -> /GPIO29
- C33 pad 1: Net-(U7-DCPL_PFD_CHP) -> GND
- C33 pad 2: GND -> Net-(C33-Pad2)
- D1 pad 1: VBUS -> +5V
- J1 pad A4: VBUS -> /VBUS
- J1 pad A9: VBUS -> /VBUS
- J1 pad B4: VBUS -> /VBUS
- J1 pad B9: VBUS -> /VBUS
- J4 pad 1: Net-(J4-In) -> GND
- J4 pad 2: GND -> +2S
- U3 pad 3: VBUS -> +5V
- U4 pad 4: /GPIO2 SDA -> /GPIO2
- U4 pad 5: /GPIO3 SCL -> /GPIO3
- U5 pad 1: /GPIO4 -> /GPIO16
- U5 pad 12: /GPIO7 -> /GPIO17
- U5 pad 13: /GPIO6 -> /GPIO18
- U5 pad 14: /GPIO5 -> /GPIO19
- U6 pad 2: /GPIO3 SCL -> /GPIO5
- U6 pad 4: /GPIO2 SDA -> /GPIO4
- U7 pad 1: +3.3VA -> GND
- U7 pad 2: /GPIO22 -> Net-(D4-A)
- U7 pad 3: /GPIO21 -> +2S
Routing:
- net VBUS: track 90.4 -> 0.00 mm
- net /RUN: track 58.6 -> 0.00 mm, vias 2 -> 0
- net /GPIO21: track 40.2 -> 0.00 mm, vias 2 -> 0
- net /GPIO22: track 39.8 -> 0.00 mm, vias 2 -> 0
- net /GPIO24: track 39.3 -> 0.00 mm, vias 2 -> 0
- net /GPIO23: track 36.5 -> 0.00 mm, vias 2 -> 0
- net /GPIO0: track 35.9 -> 0.00 mm, vias 3 -> 0
- net /SWD: track 35.3 -> 0.00 mm, vias 1 -> 0
- net /SWCLK: track 34.8 -> 0.00 mm, vias 1 -> 0
- net +3V3: track 34.3 -> 0.00 mm, vias 27 -> 0
- net /QSPI_SS: track 31.1 -> 0.00 mm, vias 2 -> 0
- net +1V1: track 30.7 -> 0.00 mm
- net /QSPI_SD1: track 29.7 -> 0.00 mm, vias 2 -> 0
- net /GPIO8: track 29.1 -> 0.00 mm
- net /GPIO9: track 27.5 -> 0.00 mm, vias 2 -> 0
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- removed copper zone on F.Cu, net +3.3VA
- removed copper zone on In2.Cu, net +3.3VA
Other:
- board size 35 x 55 mm -> 99.5 x 80 mm

Commit message: update
Parts:
- added R24: 200k, Resistor_SMD:R_0603_1608Metric, F.Cu at (460.7, 285.5)
- added R25: 1k, Resistor_SMD:R_0603_1608Metric, F.Cu at (460.2, 279.5)
- added R26: 100k, Resistor_SMD:R_0603_1608Metric, F.Cu at (460.2, 282.0)
- added R31: 100, Resistor_SMD:R_0603_1608Metric, F.Cu at (434.2, 321.2)
- added R32: 200k, Resistor_SMD:R_0603_1608Metric, F.Cu at (438.0, 325.7)
- added R33: 1k, Resistor_SMD:R_0603_1608Metric, F.Cu at (434.2, 326.2)
- added R34: 100k, Resistor_SMD:R_0603_1608Metric, F.Cu at (438.0, 322.2)
- J10: footprint Connector_Molex:Molex_Nano-Fit_105313-xx02_1x02_P2.50mm_Horizontal -> Connector_Molex:Molex_Nano-Fit_105309-xx02_1x02_P2.50mm_Vertical
- moved C33 98.3 mm to (434.5, 323.9)
- moved C32 96.3 mm to (436.5, 322.8), turned to -90 degrees

Commit message: pcb changes
Parts:
- added J2: SPI1+3V3, Connector_JST:JST_SH_BM06B-SRSS-TB_1x06-1MP_P1.00mm_Vertical, F.Cu at (415.8, 299.0)
- added J3: I2C1+3V3, Connector_JST:JST_SH_BM04B-SRSS-TB_1x04-1MP_P1.00mm_Vertical, F.Cu at (415.8, 290.0)
- added J5: UART+5V+I2C1, Connector_JST:JST_SH_BM06B-SRSS-TB_1x06-1MP_P1.00mm_Vertical, F.Cu at (415.8, 281.0)
- added J6: PYRO_1, Connector_Molex:Molex_Nano-Fit_105309-xx02_1x02_P2.50mm_Vertical, F.Cu at (425.2, 315.2)
- added J8: PWM1+6V, Connector_JST:JST_SH_BM03B-SRSS-TB_1x03-1MP_P1.00mm_Vertical, F.Cu at (450.2, 274.5)
- added J9: PWM2+6V, Connector_JST:JST_SH_BM03B-SRSS-TB_1x03-1MP_P1.00mm_Vertical, F.Cu at (450.2, 267.5)
- moved J4 121.0 mm to (441.5, 268.6)
- moved C1 65.4 mm to (431.4, 300.1)
- moved C17 65.4 mm to (431.8, 298.4)
- moved C2 65.4 mm to (433.8, 300.1)
- moved C20 65.4 mm to (433.6, 285.3)
- moved C8 65.4 mm to (435.8, 285.8)
- moved C9 65.4 mm to (435.8, 284.8)
- moved L1 65.4 mm to (435.8, 283.2)
- moved C10 65.4 mm to (434.5, 298.4)
- moved C19 65.4 mm to (439.5, 286.6)
- moved C11 65.4 mm to (437.4, 285.3)
- moved R10 65.4 mm to (438.5, 286.6)
- moved R12 65.4 mm to (432.5, 283.1)
- moved R13 65.4 mm to (433.6, 283.1)
- moved R8 65.4 mm to (433.3, 298.4)
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Routing:
- net +6V: track 0.00 -> 15.0 mm
- net GND: vias 0 -> 4
Other:
- board size 99.5 x 80 mm -> 40 x 80 mm
- board text removed: "3V3"
- board text removed: "GND"
- board text removed: "GP12"
- board text removed: "GP13"
- board text removed: "GP14"
- board text removed: "GP15"
- board text removed: "GP16"
- board text removed: "GP17"
- board text removed: "GP18"
- board text removed: "GP19"
- board text removed: "GP20"
- board text removed: "GP26"
- board text removed: "GP27"
- board text removed: "GP28"
- board text removed: "GP29"
- board text removed: "RUN"
- board text removed: "SWCLK"
- board text removed: "SWDIO"
- board text removed: "VBUS"

Commit message: pwr changes
Parts:
- added C30: 1000u, Capacitor_SMD:CP_Elec_10x10, F.Cu at (428.0, 265.8)
- added R27: 0, Resistor_SMD:R_0402_1005Metric_Pad0.72x0.64mm_HandSolder, F.Cu at (453.5, 310.2)
- added R28: 0, Resistor_SMD:R_0402_1005Metric_Pad0.72x0.64mm_HandSolder, F.Cu at (453.5, 312.2)
- added R29: 0, Resistor_SMD:R_0402_1005Metric_Pad0.72x0.64mm_HandSolder, F.Cu at (453.5, 314.2)
- added R30: 0, Resistor_SMD:R_0402_1005Metric_Pad0.72x0.64mm_HandSolder, F.Cu at (453.5, 316.2)
- added U8: 6V LDO, Package_TO_SOT_SMD:SOT-223-3_TabPin2, F.Cu at (446.9, 313.4)
- moved C6 75.2 mm to (422.6, 290.5), turned to -90 degrees
- moved R7 72.8 mm to (424.7, 290.5), turned to 0 degrees
- moved C5 70.8 mm to (420.9, 282.6), turned to 180 degrees
- moved R1 69.2 mm to (428.2, 290.5), turned to 180 degrees
- moved U2 69.0 mm to (425.0, 286.5), turned to 180 degrees
- moved R2 63.5 mm to (430.6, 287.3), turned to -90 degrees
- moved U1 63.5 mm to (425.0, 279.5), turned to 180 degrees
- moved R6 58.4 mm to (431.1, 282.2), turned to 90 degrees
- moved R3 55.6 mm to (431.1, 278.9), turned to -90 degrees
- moved C1 7.81 mm to (431.7, 307.9)
- moved C10 7.81 mm to (434.8, 306.2)
- moved C11 7.81 mm to (437.7, 293.1)
- moved C17 7.81 mm to (432.1, 306.2)
- moved C19 7.81 mm to (439.8, 294.4)
- moved C2 7.81 mm to (434.1, 307.9)
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Connections:
- U4 pad 40: /GPIO26_ADC0 -> Net-(U4-GPIO26_ADC0)
- U4 pad 41: /GPIO27_ADC1 -> Net-(U4-GPIO27_ADC1)
- U4 pad 42: /GPIO28_ADC2 -> Net-(U4-GPIO28_ADC2)
- U4 pad 43: /GPIO29_ADC3 -> Net-(U4-GPIO29_ADC3)
