File: CARP-LITE/CARP.kicad_pcb (KiCad board)
At the start: 4 copper layers, 40 x 80 mm, 89 parts, among them J1 USB_C_Receptacle_USB2.0_14P, J10 PYRO_2, J2 SPI1+3V3, J3 I2C1+3V3, J4 2S XT30, J5 UART+5V+I2C1, J6 PYRO_1, J8 PWM1+6V, J9 PWM2+6V, SW1 SW_Push, SW2 SW_Push, U1 W25Q128JVSIMTR (16MB), U2 W25Q32RVXHJQ (2MB), U3 3V3 LDO, U4 RP2350_60QFN, U5 LSM6DSO, U6 BMP390, U7 5V LDO, U8 6V LDO, Y1 ABM8-272-T3

Commit message: siup
Parts:
- added C34: 10u, Capacitor_SMD:C_0603_1608Metric, F.Cu at (465.5, 250.8)
- added C35: 10u, Capacitor_SMD:C_0603_1608Metric, F.Cu at (465.5, 253.3)
- added D2: 5V, LED_SMD:LED_0805_2012Metric, F.Cu at (469.8, 264.4)
- added Q5: SQ2318CES, Package_TO_SOT_SMD:SOT-23, F.Cu at (470.0, 251.7)
- added Q6: SQ2318CES, Package_TO_SOT_SMD:SOT-23, F.Cu at (470.0, 256.2)
- added Q7: SQ2318CES, Package_TO_SOT_SMD:SOT-23, F.Cu at (470.0, 260.6)
- added R14: 10k, Resistor_SMD:R_0603_1608Metric, F.Cu at (465.5, 255.8)
- added R15: 100, Resistor_SMD:R_0603_1608Metric, F.Cu at (465.5, 258.3)
- added R16: 5.1k, Resistor_SMD:R_0603_1608Metric, F.Cu at (465.5, 260.8)
- added R17: 100k, Resistor_SMD:R_0603_1608Metric, F.Cu at (465.5, 263.3)
- added R18: 200k, Resistor_SMD:R_0603_1608Metric, F.Cu at (465.5, 265.8)
- added R35: 100, Resistor_SMD:R_0603_1608Metric, F.Cu at (465.5, 268.3)
- R1, R11, R2, R3, R6, R7, R9: footprint PCM_Resistor_SMD_AKL:R_0603_1608Metric -> Resistor_SMD:R_0603_1608Metric
- moved C30 1.12 mm to (427.0, 266.2)

Commit message: change jst to picoblade
Parts:
- added BZ1: Buzzer, Buzzer_Beeper:Buzzer_12x9.5RM7.6, F.Cu at (398.5, 291.0)
- J5: footprint Connector_JST:JST_SH_BM06B-SRSS-TB_1x06-1MP_P1.00mm_Vertical -> Connector_Molex:Molex_PicoBlade_53047-0610_1x06_P1.25mm_Vertical
- moved J5 3.76 mm to (415.5, 277.2)

Commit message: siup
Parts:
- J2: footprint Connector_JST:JST_SH_BM06B-SRSS-TB_1x06-1MP_P1.00mm_Vertical -> Connector_Molex:Molex_PicoBlade_53047-0610_1x06_P1.25mm_Vertical
- J3: footprint Connector_JST:JST_SH_BM04B-SRSS-TB_1x04-1MP_P1.00mm_Vertical -> Connector_Molex:Molex_PicoBlade_53047-0410_1x04_P1.25mm_Vertical
- J8, J9: footprint Connector_JST:JST_SH_BM03B-SRSS-TB_1x03-1MP_P1.00mm_Vertical -> Connector_Molex:Molex_PicoBlade_53047-0310_1x03_P1.25mm_Vertical
- moved BZ1 39.1 mm to (435.4, 278.2)
- moved J2 3.34 mm to (415.0, 295.8)
- moved J3 2.24 mm to (415.0, 287.9)
- moved J5 0.56 mm to (415.0, 277.5)
