File: CARP-LITE/radio.kicad_sch (KiCad schematic)
At the start: 0 parts

Commit message: radio idk
Parts:
- added C3, C36: 100n, Capacitor_SMD:C_0603_1608Metric, symbol Device:C_Small
- added C37: 100n, symbol Device:C_Small
- added C38: 18p, symbol Device:C_Small
- added C39, C45: 470p, Capacitor_SMD:C_0402_1005Metric, symbol Device:C_Small
- added C4, C53, C54, C56, C57: 4.7u, Capacitor_SMD:C_0603_1608Metric, symbol Device:C_Small
- added C40: 6.8p, Capacitor_SMD:C_0402_1005Metric, symbol Device:C_Small
- added C41: 2.7p, Capacitor_SMD:C_0402_1005Metric, symbol Device:C_Small
- added C42: 1.1p, Capacitor_SMD:C_0402_1005Metric, symbol Device:C_Small
- added C43: 1.2p, Capacitor_SMD:C_0402_1005Metric, symbol Device:C_Small
- added C44: 2.0p, Capacitor_SMD:C_0402_1005Metric, symbol Device:C_Small
- added C46: 11p, Capacitor_SMD:C_0402_1005Metric, symbol Device:C_Small
- added C47: 22p, Capacitor_SMD:C_0402_1005Metric, symbol Device:C_Small
- added C48: 5.6p, Capacitor_SMD:C_0402_1005Metric, symbol Device:C_Small
- added C49: 18p, Capacitor_SMD:C_0402_1005Metric, symbol Device:C_Small
- added C50, C55: 10p, Capacitor_SMD:C_0402_1005Metric, symbol Device:C_Small
- added C51: 1.6p, Capacitor_SMD:C_0402_1005Metric, symbol Device:C_Small
- added C52: 47p, Capacitor_SMD:C_0402_1005Metric, symbol Device:C_Small
- added FB1, FB2, FB3: 50@100M, Inductor_SMD:L_0603_1608Metric, symbol Device:FerriteBead_Small
- added J11: RF_L, Connector_Coaxial:U.FL_Hirose_U.FL-R-SMT-1_Vertical, symbol Connector:Conn_Coaxial_Small
- added J7: RF_H, Connector_Coaxial:U.FL_Hirose_U.FL-R-SMT-1_Vertical, symbol Connector:Conn_Coaxial_Small
- added L10: 5.1n, Inductor_SMD:L_0402_1005Metric, symbol Device:L_Small
- added L11: 7.5n, Inductor_SMD:L_0402_1005Metric, symbol Device:L_Small
- added L12: 27n, Inductor_SMD:L_0402_1005Metric, symbol Device:L_Small
- added L13: 75n, Inductor_SMD:L_0402_1005Metric, symbol Device:L_Small
- added L2: 4.7u, Inductor_SMD:L_0805_2012Metric, symbol Device:L_Small
- added L3: 2.4n, Inductor_SMD:L_0402_1005Metric, symbol Device:L_Small
- added L4: 18n, Inductor_SMD:L_0402_1005Metric, symbol Device:L_Small
- added L5: 1.5n, Inductor_SMD:L_0402_1005Metric, symbol Device:L_Small
- added L6: 1.9n, Inductor_SMD:L_0402_1005Metric, symbol Device:L_Small
- added L7: 1.1n, Inductor_SMD:L_0402_1005Metric, symbol Device:L_Small
- added L8: 22n, Inductor_SMD:L_0402_1005Metric, symbol Device:L_Small
- added L9: 10n, Inductor_SMD:L_0402_1005Metric, symbol Device:L_Small
- added U9: LR2021IMLTRT, Package_DFN_QFN:QFN-32-1EP_5x5mm_P0.5mm_EP3.7x3.7mm_ThermalVias, symbol Radio:LR2021
- added Y2: TG2520SMN-32.0000M-MCGNNM0, Oscillator:Oscillator_SMD_ECS_2520MV-xxx-xx-4Pin_2.5x2.0mm, symbol Oscillator:TG2520SMN-xx.xxxxxxMhz-xxxxNM
Connections:
- new net: C40.1, C41.1, C42.1, L6.1
- new net: C40.2, L5.2
- new net: C50.1, C52.1, J11.1 (In), L11.2, L12.1
- new net: C38.1, L3.2
- new net: C38.2, C42.2, C43.1, L6.2, L7.1
- new net: C3.1, C4.1, FB3.1, U9.17 (VBAT)
- new net: C56.1, FB2.1, U9.12 (VDCC1)
- new net: C48.2, C49.1, L10.2, L11.1
- new net: C44.1, J7.1 (In), L7.2
- new net: C57.1, FB2.2, U9.26 (VDCC2)
- new net: C54.1, FB1.1, U9.13 (VPAX1)
- new net: C46.2, L9.2
- new net: C46.1, C47.1, C48.1, L10.1
- new net: C53.1, FB1.2, U9.2 (VPAX2)
- new net: C51.1, C52.2, L13.2
- new net: C55.2, Y2.3 (OUT)
- new net: L2.1, U9.16 (LXA)
- new net: L2.2, U9.14 (LXB)
- new net +3V3: FB3.2
- new net GND: C3.2, C36.2, C37.1, C39.1, C4.2, C41.2, C43.2, C44.2, C45.1, C47.2, C49.2, C50.2, C51.2, C53.2, C54.2, C56.2, C57.2, J11.2 (Ext), J7.2 (Ext), L12.2, U9.15 (GND_DCC), U9.30 (GND), U9.33 (GND), Y2.2 (GND)
- new net RADIO_BUSY: U9.25 (BUSY)
- new net RADIO_CS: U9.24 (CS)
- new net RADIO_DIO5: U9.19 (DIO5)
- new net RADIO_DIO6: U9.18 (DIO6)
- new net RADIO_MISO: U9.21 (MISO)
- new net RADIO_MOSI: U9.22 (MOSI)
- new net RADIO_SCK: U9.23 (SCK)
- new net RFI_HF: L3.1, U9.31 (RFI_HF)
- new net RFI_LF: L13.1, U9.29 (RFI_LF)
- new net RFO_HF: L4.2, L5.1, U9.32 (RFO_HF)
- new net RFO_LF1: L8.2, L9.1, U9.27 (RFO_LF2), U9.28 (RFO_LF1)
- new net TCXO_CLK: C55.1, U9.4 (XTA)
- new net VR_PA: C36.1, C39.2, C45.2, L4.1, L8.1, U9.1 (VR_PA)
- new net VTCXO: C37.2, U9.6 (VTCXO/VNTC), Y2.4 (Vcc)
- new net ~{RADIO_RESET}: U9.20 (~{RESET})
- no-connect marks 0 -> 7
Other:
- note added: "What The Fuck"

Commit message: Forgor to save oops
Parts:
- FB1, FB2: value 50@100M -> 60@100M; MFR (none) -> ILHB0603ER600V
- FB3: MFR (none) -> ILHB0603ER600V
- L2: MFR (none) -> IMC2220ER4R7K
Changed lines of the file:
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@@
+	)
+	(symbol
+		(lib_id "Device:FerriteBead_Small")
+		(at 171.45 52.07 90)
+		(unit 1)
+		(body_style 1)
+		(exclude_from_sim no)
+		(in_bom yes)
+		(on_board yes)
+		(in_pos_files yes)
+		(dnp no)
+		(property "Reference" "FB1"
+			(at 171.45 45.212 90)
+			(show_name no)
+			(do_not_autoplace no)
+			(effects
+				(font
+					(size 1.27 1.27)
+				)
+			)
+		)
+		(property "Value" "60@100M"
+			(at 171.45 47.752 90)
+			(show_name no)
+			(do_not_autoplace no)
+			(effects
+				(font
+					(size 1.27 1.27)
+				)
+			)
+		)
+		(property "Footprint" "Inductor_SMD:L_0603_1608Metric"
+			(at 171.45 53.848 90)
+			(hide yes)
+			(show_name no)
+			(do_not_autoplace no)
+			(effects
+				(font
+					(size 1.27 1.27)
+				)
+			)
+		)
+		(property "Datasheet" ""
+			(at 171.45 52.07 0)
+			(hide yes)
+			(show_name no)
+			(do_not_autoplace no)
+			(effects
+				(font
+					(size 1.27 1.27)
+				)
+			)
+		)
+		(property "Description" "Ferrite bead, small symbol"
+			(at 171.45 52.07 0)
+			(hide yes)
+			(show_name no)
+			(do_not_autoplace no)
+			(effects
+				(font
+					(size 1.27 1.27)
+				)
+			)
+		)
+		(property "MFR" "ILHB0603ER600V"
+			(at 171.45 52.07 90)
+			(hide yes)
+			(show_name no)
+			(do_not_autoplace no)
+			(effects
+				(font
+					(size 1.27 1.27)
+				)
+			)
+		)
+		(pin "2"
+		)
+		(pin "1"
+		)
+		(instances
+			(project "CARP"
+				(path "/94683f5c-9cd9-448e-be96-9792537b5cb8/fbf78cf6-1e60-4f5c-8e3f-17a0841f8e52"
+					(reference "FB1")
+					(unit 1)
+				)
+			)
+		)
 	)
 	(symbol
@@
 			)
 		)
-		(property "Value" "50@100M"
+		(property "Value" "60@100M"
 			(at 147.32 48.006 90)
 			(show_name no)
@@
 		(property "Description" "Ferrite bead, small symbol"
 			(at 147.32 57.15 0)
+			(hide yes)
+			(show_name no)
+			(do_not_autoplace no)
+			(effects
+				(font
+					(size 1.27 1.27)
+				)
+			)
+		)
+		(property "MFR" "ILHB0603ER600V"
+			(at 147.32 57.15 90)
 			(hide yes)
 			(show_name no)
@@
 			)
 		)
+		(property "MFR" "ILHB0603ER600V"
+			(at 138.43 76.2 90)
+			(hide yes)
+			(show_name no)
+			(do_not_autoplace no)
+			(effects
+				(font
+					(size 1.27 1.27)
+				)
+			)
+		)
 		(pin "2"
 		)
@@
 	)
 	(symbol
-		(lib_id "Device:FerriteBead_Small")
-		(at 171.45 52.07 90)
-		(unit 1)
-		(body_style 1)
-		(exclude_from_sim no)
-		(in_bom yes)
-		(on_board yes)
-		(in_pos_files yes)
-		(dnp no)
-		(fields_autoplaced yes)
-		(property "Reference" "FB1"
-			(at 171.4119 45.72 90)
-			(show_name no)
-			(do_not_autoplace no)
-			(effects
-				(font
-					(size 1.27 1.27)
-				)
-			)
-		)
-		(property "Value" "50@100M"
-			(at 171.4119 48.26 90)
-			(show_name no)
-			(do_not_autoplace no)
-			(effects
-				(font
-					(size 1.27 1.27)
-				)
-			)
-		)
-		(property "Footprint" "Inductor_SMD:L_0603_1608Metric"
-			(at 171.45 53.848 90)
-			(hide yes)
-			(show_name no)
-			(do_not_autoplace no)
-			(effects
-				(font
-					(size 1.27 1.27)
-				)
-			)
-		)
-		(property "Datasheet" ""
-			(at 171.45 52.07 0)
-			(hide yes)
-			(show_name no)
-			(do_not_autoplace no)
-			(effects
-				(font
-					(size 1.27 1.27)
-				)
-			)
-		)
-		(property "Description" "Ferrite bead, small symbol"
-			(at 171.45 52.07 0)
-			(hide yes)
-			(show_name no)
-			(do_not_autoplace no)
-			(effects
-				(font
-					(size 1.27 1.27)
-				)
-			)
-		)
-		(pin "2"
-		)
-		(pin "1"
-		)
-		(instances
-			(project "CARP"
-				(path "/94683f5c-9cd9-448e-be96-9792537b5cb8/fbf78cf6-1e60-4f5c-8e3f-17a0841f8e52"
-					(reference "FB1")
-					(unit 1)
-				)
-			)
-		)
-	)
-	(symbol
 		(lib_id "power:GND")
 		(at 255.27 77.47 0)
@@
 			(at 127 68.58 0)
 			(hide yes)
+			(show_name no)
+			(do_not_autoplace no)
+			(effects
+				(font
+					(size 1.27 1.27)
+				)
+			)
+		)
+		(property "MFR" "IMC2220ER4R7K"
+			(at 127 68.58 0)
+			(hide yes)

Commit message: Update button footprint to proper one
Other:
- company: (none) -> Silesian Aerospace Technologies
- title: (none) -> CARP-LITE
Changed lines of the file:
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@@
 	(generator_version "10.0")
 	(paper "A4")
+	(title_block
+		(title "CARP-LITE")
+		(date "2026-06-29")
+		(rev "V1")
+		(company "Silesian Aerospace Technologies")
+		(comment 1 "Marcin Czop")
+		(comment 2 "Aria Wiktoria Horak")
+	)
 	(rectangle
 		(start 186.69 13.97)

Commit message: fp cahnges
Parts:
- C37: footprint (none) -> Capacitor_SMD:C_0603_1608Metric
- C38: footprint (none) -> Capacitor_SMD:C_0402_1005Metric
Changed lines of the file:
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@@
 			)
 		)
-		(property "Footprint" ""
+		(property "Footprint" "Capacitor_SMD:C_0603_1608Metric"
 			(at 227.33 127 0)
 			(hide yes)
@@
 			)
 		)
-		(property "Footprint" ""
+		(property "Footprint" "Capacitor_SMD:C_0402_1005Metric"
 			(at 219.71 49.53 0)
 			(hide yes)

Commit message: update inductor
Parts:
- L2: footprint Inductor_SMD:L_0805_2012Metric -> Inductor_SMD:L_1008_2520Metric; MFR IMC2220ER4R7K -> 1008AF-472XJRC
Changed lines of the file:
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@@
 			)
 		)
-		(property "Footprint" "Inductor_SMD:L_0805_2012Metric"
+		(property "Footprint" "Inductor_SMD:L_1008_2520Metric"
 			(at 127 68.58 0)
 			(hide yes)
@@
 			)
 		)
-		(property "MFR" "IMC2220ER4R7K"
+		(property "MFR" "1008AF-472XJRC"
 			(at 127 68.58 0)
 			(hide yes)

Commit message: update values
Parts:
- L5: value 1.5n -> 1.7n
- L7: value 1.1n -> 1n
Changed lines of the file:
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@@
 			)
 		)
-		(property "Value" "1.5n"
+		(property "Value" "1.7n"
 			(at 217.17 34.29 90)
 			(show_name no)
@@
 			)
 		)
-		(property "Value" "1.1n"
+		(property "Value" "1n"
 			(at 252.73 34.29 90)
 			(show_name no)

Commit message: change sizes
Parts:
- Y2: value TG2520SMN-32.0000M-MCGNNM0 -> ECS-TXO-25CSMV-320-AN-TR
Changed lines of the file:
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@@
 			)
 		)
-		(property "Value" "TG2520SMN-32.0000M-MCGNNM0"
+		(property "Value" "ECS-TXO-25CSMV-320-AN-TR"
 			(at 224.79 137.1599 0)
 			(show_name no)
