File: CARP-LITE/rev2.0/lithium_charger.kicad_sch (KiCad schematic)
At the start: 23 parts, among them U1 BQ25792

Commit message: update revision on schematics
Other:
- company: (none) -> Silesian Aerospace Technologies
- title: (none) -> CARP-LITE
Changed lines of the file:
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@@
 	(generator_version "10.0")
 	(paper "A4")
+	(title_block
+		(title "CARP-LITE")
+		(date "2026-09-07")
+		(rev "V2")
+		(company "Silesian Aerospace Technologies")
+		(comment 1 "Aria Wiktoria Horak")
+	)
 	(junction
 		(at 172.72 66.04)
