File: CARP-LITE/rev2.0/radio.kicad_sch (KiCad schematic)
At the start: 43 parts, among them J11 RF_L, J7 RF_H, U9 LR2021IMLTRT, Y2 ECS-TXO-25CSMV-320-AN-TR

Commit message: rev 2 schematic changes
Parts:
- removed C38: 18p, Capacitor_SMD:C_0402_1005Metric, symbol Device:C_Small
- removed C39: 470p, Capacitor_SMD:C_0402_1005Metric, symbol Device:C_Small
- removed C40: 6.8p, Capacitor_SMD:C_0402_1005Metric, symbol Device:C_Small
- removed C41: 2.7p, Capacitor_SMD:C_0402_1005Metric, symbol Device:C_Small
- removed C42: 1.1p, Capacitor_SMD:C_0402_1005Metric, symbol Device:C_Small
- removed C43: 1.2p, Capacitor_SMD:C_0402_1005Metric, symbol Device:C_Small
- removed C44: 2.0p, Capacitor_SMD:C_0402_1005Metric, symbol Device:C_Small
- removed J7: RF_H, Connector_Coaxial:U.FL_Hirose_U.FL-R-SMT-1_Vertical, symbol Connector:Conn_Coaxial_Small
- removed L3: 2.4n, Inductor_SMD:L_0402_1005Metric, symbol Device:L_Small
- removed L4: 18n, Inductor_SMD:L_0402_1005Metric, symbol Device:L_Small
- removed L5: 1.7n, Inductor_SMD:L_0402_1005Metric, symbol Device:L_Small
- removed L6: 1.9n, Inductor_SMD:L_0402_1005Metric, symbol Device:L_Small
- removed L7: 1n, Inductor_SMD:L_0402_1005Metric, symbol Device:L_Small
- C3, C36, C37: footprint Capacitor_SMD:C_0603_1608Metric -> Capacitor_SMD:C_0402_1005Metric
Connections:
- net RFI_HF: no longer names the net of U9.31 (RFI_HF)
- net RFO_HF: no longer names the net of U9.32 (RFO_HF)
- no-connect marks 7 -> 9
Other:
- note added: "32MHz TCXO"
- note added: "433MHz matching network"
- note removed: "What The Fuck"
- moved on the sheet: C36, C37, C45, C46, C47, C48, C49, C50, C51, C52, C55, J11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

Commit message: radio dosen't need two interrupts
Connections:
- net RADIO_DIO6: no longer names the net of U9.18 (DIO6)
- no-connect marks 9 -> 10
Changed lines of the file:
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@@
+	)
+	(no_connect
+		(at 95.25 43.18)
 	)
 	(no_connect
@@
 	(wire
 		(pts
-			(xy 83.82 43.18) (xy 95.25 43.18)
-		)
-		(stroke
-			(width 0)
-			(type default)
-		)
-	)
-	(wire
-		(pts
 			(xy 243.84 36.83) (xy 241.3 36.83)
 		)
@@
 		(pts
 			(xy 226.06 36.83) (xy 233.68 36.83)
-		)
-		(stroke
-			(width 0)
-			(type default)
-		)
-	)
-	(wire
-		(pts
-			(xy 27.94 45.72) (xy 39.37 45.72)
 		)
 		(stroke
@@
 		)
 	)
-	(label "DIO6"
-		(at 27.94 45.72 0)
-		(effects
-			(font
-				(size 1.27 1.27)
-			)
-			(justify left bottom)
-		)
-	)
 	(label "BUSY"
 		(at 27.94 53.34 0)
-		(effects
-			(font
-				(size 1.27 1.27)
-			)
-			(justify left bottom)
-		)
-	)
-	(label "DIO6"
-		(at 83.82 43.18 0)
 		(effects
 			(font
@@
 		(effects
 			(font
-				(size 1.27 1.27)
-			)
-			(justify left)
-		)
-	)
-	(hierarchical_label "RADIO_DIO6"
-		(shape bidirectional)
-		(at 39.37 45.72 0)
-		(effects
-			(font
