File: CARP-LITE/rev2.0/CARP.kicad_sch (KiCad schematic)
At the start: 110 parts, among them J1 USB-C, J10 PYRO_2, J3 I2C1+3V3, J4 2S XT30, J5 UART+5V+I2C1, J6 PYRO_1, J8 PWM1+5V1, J9 PWM2+5V1, Q5 SQ2318CES, Q6 SQ2318CES, Q7 SQ2318CES, SW1 SW_Push, SW2 SW_Push, U1 W25Q128JVSIMTR (16MB), U10 TPS62130A, U2 W25Q32RVXHJQ (2MB), U4 RP2350_60QFN, U5 LSM6DSO, U6 BMP390, U7 TLV75733PDBV, Y1 ABM8-272-T3

Commit message: adjust silkscreen
Parts:
- C31, C32: value 100n -> 1n
Changed lines of the file:
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@@
 		)
 	)
+	(text_box "change notes:\n\n- c32, c31 changed from 100n to 1n (held charge too long)"
+		(exclude_from_sim no)
+		(at 240.03 182.88 0)
+		(size 45.72 54.61)
+		(margins 0.9525 0.9525 0.9525 0.9525)
+		(stroke
+			(width 0)
+			(type solid)
+		)
+		(fill
+			(type none)
+		)
+		(effects
+			(font
+				(size 1.27 1.27)
+			)
+			(justify left top)
+		)
+	)
 	(junction
 		(at 57.15 88.9)
@@
 			)
 		)
-		(property "Value" "100n"
+		(property "Value" "1n"
 			(at 322.072 222.758 0)
 			(show_name no)
@@
 			)
 		)
-		(property "Value" "100n"
+		(property "Value" "1n"
 			(at 322.072 185.928 0)
 			(show_name no)

Commit message: rev 2 schematic changes
Parts:
- removed C5: 100n, Capacitor_SMD:C_0402_1005Metric, symbol Device:C
- removed R3: 0, Resistor_SMD:R_0603_1608Metric, symbol Device:R
- removed R6: 5.1k, Resistor_SMD:R_0402_1005Metric, symbol Device:R
- removed U1: W25Q128JVSIMTR (16MB), Package_SO:SOIC-8_5.3x5.3mm_P1.27mm, symbol Memory_Flash:W25Q128JVS
- U2: value W25Q32RVXHJQ (2MB) -> W25Q128JVSIMTR (16MB)
Other:
- note removed: "Flight Data Flash"

Commit message: radio dosen't need two interrupts
Other:
- sheet Radio ports: added none; removed RADIO_DIO6
Changed lines of the file:
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@@
 	(text "Radio\n"
 		(exclude_from_sim no)
-		(at 230.632 282.448 0)
+		(at 230.124 282.194 0)
 		(effects
 			(font
@@
 	(wire
 		(pts
-			(xy 238.76 273.05) (xy 248.92 273.05)
+			(xy 237.49 270.51) (xy 247.65 270.51)
 		)
 		(stroke
@@
 	(wire
 		(pts
-			(xy 238.76 257.81) (xy 248.92 257.81)
-		)
-		(stroke
-			(width 0)
-			(type default)
-		)
-	)
-	(wire
-		(pts
 			(xy 87.63 41.91) (xy 87.63 43.18)
 		)
@@
 	(wire
 		(pts
-			(xy 238.76 264.16) (xy 248.92 264.16)
+			(xy 237.49 259.08) (xy 247.65 259.08)
 		)
 		(stroke
@@
 	(wire
 		(pts
+			(xy 237.49 264.16) (xy 247.65 264.16)
+		)
+		(stroke
+			(width 0)
+			(type default)
+		)
+	)
+	(wire
+		(pts
 			(xy 205.74 248.92) (xy 209.55 248.92)
 		)
@@
 	(wire
 		(pts
+			(xy 237.49 261.62) (xy 247.65 261.62)
+		)
+		(stroke
+			(width 0)
+			(type default)
+		)
+	)
+	(wire
+		(pts
 			(xy 127 81.28) (xy 134.62 81.28)
 		)
@@
 	(wire
 		(pts
-			(xy 238.76 270.51) (xy 248.92 270.51)
+			(xy 237.49 267.97) (xy 247.65 267.97)
 		)
 		(stroke
@@
 	(wire
 		(pts
-			(xy 238.76 266.7) (xy 248.92 266.7)
-		)
-		(stroke
-			(width 0)
-			(type default)
-		)
-	)
-	(wire
-		(pts
 			(xy 321.31 43.18) (xy 321.31 55.88)
 		)
@@
 	(wire
 		(pts
-			(xy 238.76 278.13) (xy 248.92 278.13)
+			(xy 237.49 275.59) (xy 247.65 275.59)
 		)
 		(stroke
@@
 	(wire
 		(pts
-			(xy 238.76 260.35) (xy 248.92 260.35)
-		)
-		(stroke
-			(width 0)
-			(type default)
-		)
-	)
-	(wire
-		(pts
 			(xy 311.15 200.66) (xy 325.12 200.66)
 		)
@@
 	(wire
 		(pts
-			(xy 238.76 275.59) (xy 248.92 275.59)
+			(xy 237.49 273.05) (xy 247.65 273.05)
 		)
 		(stroke
@@
 				)
 			)
-			(table_cell "RADIO DIO6"
+			(table_cell ""
 				(exclude_from_sim no)
 				(at 369.57 193.04 0)
@@
 	)
 	(label "GPIO15"
-		(at 238.76 273.05 0)
+		(at 237.49 270.51 0)
 		(effects
 			(font
@@
 	)
 	(label "GPIO10"
-		(at 238.76 260.35 0)
+		(at 237.49 261.62 0)
 		(effects
 			(font
@@
 	)
 	(label "GPIO14"
-		(at 238.76 278.13 0)
+		(at 237.49 275.59 0)
 		(effects
 			(font
@@
 	)
 	(label "GPIO11"
-		(at 238.76 257.81 0)
+		(at 237.49 259.08 0)
 		(effects
 			(font
@@
 	)
 	(label "GPIO13"
-		(at 238.76 275.59 0)
-		(effects
-			(font
-				(size 1.27 1.27)
-			)
-			(justify left bottom)
-		)
-	)
-	(label "GPIO7"
-		(at 238.76 266.7 0)
+		(at 237.49 273.05 0)
 		(effects
 			(font
@@
 	)
 	(label "GPIO12"
-		(at 238.76 270.51 0)
+		(at 237.49 267.97 0)
 		(effects
 			(font
@@
 	)
 	(label "GPIO6"
-		(at 238.76 264.16 0)
+		(at 237.49 264.16 0)
 		(effects
 			(font
@@
 	)
 	(sheet
-		(at 248.92 256.54)
-		(size 15.24 22.86)
+		(at 247.65 257.81)
+		(size 15.24 19.05)
 		(exclude_from_sim no)
 		(in_bom yes)
@@
 		)
 		(property "Sheetname" "Radio"
-			(at 248.92 255.8284 0)
+			(at 247.65 257.0984 0)
 			(show_name no)
 			(do_not_autoplace no)
@@
 		)
 		(property "Sheetfile" "radio.kicad_sch"
-			(at 248.92 279.9846 0)
+			(at 247.65 277.4446 0)
 			(show_name no)
 			(do_not_autoplace no)
@@
 		)
 		(pin "RADIO_BUSY" input
-			(at 248.92 260.35 180)
+			(at 247.65 261.62 180)
 			(effects
 				(font
@@
 		)
 		(pin "RADIO_CS" input
-			(at 248.92 275.59 180)
+			(at 247.65 273.05 180)
 			(effects
 				(font
@@
 		)
 		(pin "RADIO_DIO5" bidirectional
-			(at 248.92 264.16 180)
-			(effects
-				(font
-					(size 1.27 1.27)
-				)
-				(justify left)
-			)
-		)
-		(pin "RADIO_DIO6" bidirectional
-			(at 248.92 266.7 180)
+			(at 247.65 264.16 180)
 			(effects
 				(font
@@
 		)
 		(pin "RADIO_MISO" output
-			(at 248.92 270.51 180)
+			(at 247.65 267.97 180)
 			(effects
 				(font
@@
 		)
 		(pin "RADIO_MOSI" input
-			(at 248.92 273.05 180)
+			(at 247.65 270.51 180)
 			(effects
 				(font
@@
 		)
 		(pin "RADIO_SCK" input
-			(at 248.92 278.13 180)
+			(at 247.65 275.59 180)
 			(effects
 				(font
@@
 		)
 		(pin "~{RADIO_RESET}" input
-			(at 248.92 257.81 180)
+			(at 247.65 259.08 180)
 			(effects
 				(font

Commit message: more rev2 schematic stuff
Parts:
- added J7: SPI, Connector_Molex:Molex_PicoBlade_53047-0610_1x06_P1.25mm_Vertical, symbol Connector_Generic:Conn_01x06
Connections:
- net +5V: now also J7.6 (Pin_6)
- net GND: now also J7.1 (Pin_1)
- net GPIO12: now also J7.5 (Pin_5)
- net GPIO14: now also J7.3 (Pin_3)
- net GPIO15: now also J7.4 (Pin_4)
- net GPIO25: now also J7.2 (Pin_2); no longer D1.4 (DIN)
- net GPIO6: now also U5.4 (INT1)
- new net GPIO1: D1.4 (DIN)

Commit message: 2/3S Lithium Cell Charger
Parts:
- removed D3: V2FL45, Diode_SMD:D_SMF, symbol Device:D_Schottky
- removed D4: VSSAF5L45, Diode_SMD:D_SMA, symbol Device:D_Schottky
- removed R1: DNF, Resistor_SMD:R_0603_1608Metric, symbol Device:R
- J4: value 2S XT30 -> 2/3S XT30
Connections:
- net +2S: no longer C60.2, J4.2 (Pin_2), U10.10 (VIN), U10.11 (VIN), U10.12 (VIN), U10.13 (EN)
- net +5V: now also C58.1, C61.1, C62.1, L14.2, R23.1, R36.1, TP1.1, U10.14 (VOS)
- net +5V1: no longer C58.1, C61.1, C62.1, L14.2, R23.1, R36.1, TP1.1, U10.14 (VOS)
- new net BAT: J4.2 (Pin_2)
- new net CHRGR_OUT: C60.2, U10.10 (VIN), U10.11 (VIN), U10.12 (VIN), U10.13 (EN)
Other:
- added sheet Lithium Charger (lithium_charger.kicad_sch)
- moved on the sheet: C26, C29, C58, C59, C60, C61, C62, D2, L14, R16, R17, R18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

Commit message: IMU interrupt GPIO fix
Connections:
- net GPIO6: no longer U5.4 (INT1)
- net GPIO7: now also U5.4 (INT1)
Changed lines of the file:
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@@
 		)
 	)
-	(label "GPIO6"
+	(label "GPIO7"
 		(at 115.57 212.09 0)
 		(effects

Commit message: Replace baro with BMP581 and some small changes
Parts:
- removed U6: BMP390, bmp_fps:10LGA_2X2X0p75_BOS, symbol 2026-03-13_01-43-10:BMP390
- added U3: BMP581, bmp_fps:10LGA_2X2X0p75_BOS, symbol BMP581:BMP581
Connections:
- net +2S: no longer J10.1 (Pin_1), J6.1 (Pin_1)
- net +3V3: now also C22.1, C24.1, U3.1 (VDDIO), U3.10 (VDD), U3.5 (SDO), U3.6 (CSB); no longer C22.2, C24.2
- net BAT: now also J10.1 (Pin_1), J6.1 (Pin_1)
- net GND: now also C22.2, C24.2, U3.3 (GND), U3.8 (GND), U3.9 (GND); no longer C22.1, C24.1
- net GPIO0: now also U3.7 (INT)
- net GPIO1: now also U4.3 (GPIO1)
- net GPIO4: now also U3.4 (SDI)
- net GPIO5: now also U3.2 (SCK)
- no-connect marks 8 -> 7
Other:
- note added: "BMP581 [I2C0]"
- note added: "Default address: 0x47"
- note added: "Firmware and Flight Data Flash"
- note removed: "BMP390 [I2C0]"
- note removed: "Default address: 0x76"
- note removed: "Primary Flash"
- moved on the sheet: C25, C6, R7, TP2
