File: CARP-LITE/rev2.0/CARP.kicad_sch (KiCad schematic)
At the start: 104 parts, among them J1 USB-C, J10 PYRO_2, J3 I2C1+3V3, J4 2/3S XT30, J5 UART+5V+I2C1, J6 PYRO_1, J7 SPI, J8 PWM1+5V1, J9 PWM2+5V1, Q5 SQ2318CES, Q6 SQ2318CES, Q7 SQ2318CES, SW1 SW_Push, SW2 SW_Push, U10 TPS62130A, U2 W25Q128JVSIMTR (16MB), U3 BMP581, U4 RP2350_60QFN, U5 LSM6DSO, U7 TLV75733PDBV, Y1 ABM8-272-T3

Commit message: mess up pcb a bit
Connections:
- net +5V1 is gone; now on net +5V: C35.1, C63.1, J8.3 (Pin_3), J9.3 (Pin_3), U10.7 (FSW)
