File: Hardware/CARP-LITE/rev2.0/CARP.kicad_sch (KiCad schematic)
At the start: 104 parts, among them J1 USB-C, J10 PYRO_2, J3 I2C1+3V3, J4 2/3S XT30, J5 UART+5V+I2C1, J6 PYRO_1, J7 SPI, J8 PWM1+5V1, J9 PWM2+5V1, Q5 SQ2318CES, Q6 SQ2318CES, Q7 SQ2318CES, SW1 SW_Push, SW2 SW_Push, U10 TPS62130A, U2 W25Q128JVSIMTR (16MB), U3 BMP581, U4 RP2350_60QFN, U5 LSM6DSO, U7 TLV75733PDBV, Y1 ABM8-272-T3

Commit message: pcb and schematic changes
Connections:
- net +2S is gone; now on net BAT: R18.2
Changed lines of the file:
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@@
 	)
 	(junction
-		(at 57.15 88.9)
-		(diameter 0)
-		(color 0 0 0 0)
-	)
-	(junction
 		(at 337.82 26.67)
 		(diameter 0)
@@
 	)
 	(junction
+		(at 57.15 88.9)
+		(diameter 0)
+		(color 0 0 0 0)
+	)
+	(junction
 		(at 314.96 38.1)
 		(diameter 0)
@@
 	(wire
 		(pts
-			(xy 57.15 88.9) (xy 59.69 88.9)
-		)
-		(stroke
-			(width 0)
-			(type default)
-		)
-	)
-	(wire
-		(pts
 			(xy 303.53 27.94) (xy 303.53 26.67)
 		)
@@
 	(wire
 		(pts
+			(xy 88.9 104.14) (xy 92.71 104.14)
+		)
+		(stroke
+			(width 0)
+			(type default)
+		)
+	)
+	(wire
+		(pts
 			(xy 46.99 38.1) (xy 46.99 40.64)
 		)
@@
 	(wire
 		(pts
-			(xy 45.72 81.28) (xy 52.07 81.28)
+			(xy 45.72 81.28) (xy 54.61 81.28)
 		)
 		(stroke
@@
 	)
 	(label "VBUS"
-		(at 52.07 81.28 180)
+		(at 54.61 81.28 180)
 		(effects
 			(font
@@
 		)
 	)
+	(label "BAT"
+		(at 88.9 104.14 0)
+		(effects
+			(font
+				(size 1.27 1.27)
+			)
+			(justify left bottom)
+		)
+	)
 	(label "GPIO15"
 		(at 351.79 111.76 180)
@@
 	)
 	(symbol
-		(lib_id "power:+8V")
-		(at 92.71 104.14 0)
-		(unit 1)
-		(body_style 1)
-		(exclude_from_sim no)
-		(in_bom yes)
-		(on_board yes)
-		(in_pos_files yes)
-		(dnp no)
-		(fields_autoplaced yes)
-		(property "Reference" "#PWR058"
-			(at 92.71 107.95 0)
-			(hide yes)
-			(show_name no)
-			(do_not_autoplace no)
-			(effects
-				(font
-					(size 1.27 1.27)
-				)
-			)
-		)
-		(property "Value" "+2S"
-			(at 92.71 100.33 0)
-			(show_name no)
-			(do_not_autoplace no)
-			(effects
-				(font
-					(size 1.27 1.27)
-				)
-			)
-		)
-		(property "Footprint" ""
-			(at 92.71 104.14 0)
-			(hide yes)
-			(show_name no)
-			(do_not_autoplace no)
-			(effects
-				(font
-					(size 1.27 1.27)
-				)
-			)
-		)
-		(property "Datasheet" ""
-			(at 92.71 104.14 0)
-			(hide yes)
-			(show_name no)
-			(do_not_autoplace no)
-			(effects
-				(font
-					(size 1.27 1.27)
-				)
-			)
-		)
-		(property "Description" "Power symbol creates a global label with name \"+8V\""
-			(at 92.71 104.14 0)
-			(hide yes)
-			(show_name no)
-			(do_not_autoplace no)
-			(effects
-				(font
-					(size 1.27 1.27)
-				)
-			)
-		)
-		(pin "1"
-		)
-		(instances
-			(project "CARP"
-				(path "/94683f5c-9cd9-448e-be96-9792537b5cb8"
-					(reference "#PWR058")
-					(unit 1)
-				)
-			)
-		)
-	)
-	(symbol
 		(lib_id "Device:R")
 		(at 250.825 85.09 270)
@@
 	(symbol
 		(lib_id "power:GND")
-		(at 59.69 88.9 0)
+		(at 57.15 88.9 0)
 		(unit 1)
 		(body_style 1)
@@
 		(dnp no)
 		(property "Reference" "#PWR07"
-			(at 59.69 95.25 0)
+			(at 57.15 95.25 0)
 			(hide yes)
 			(show_name no)
@@
 		)
 		(property "Value" "GND"
-			(at 63.754 90.932 0)
+			(at 61.214 90.932 0)
 			(show_name no)
 			(do_not_autoplace no)
@@
 		)
 		(property "Footprint" ""
-			(at 59.69 88.9 0)
+			(at 57.15 88.9 0)
 			(hide yes)
 			(show_name no)
@@
 		)
 		(property "Datasheet" ""
-			(at 59.69 88.9 0)
+			(at 57.15 88.9 0)
 			(hide yes)
 			(show_name no)
@@
 		)
 		(property "Description" ""
-			(at 59.69 88.9 0)
+			(at 57.15 88.9 0)
 			(show_name no)
 			(do_not_autoplace no)

Commit message: powersection
Parts:
- C23, C59: footprint Capacitor_SMD:C_0603_1608Metric -> Capacitor_SMD:C_0402_1005Metric
- R36, R37: footprint Resistor_SMD:R_0603_1608Metric -> Resistor_SMD:R_0402_1005Metric
Changed lines of the file:
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@@
 			)
 		)
-		(property "Footprint" "Resistor_SMD:R_0603_1608Metric"
+		(property "Footprint" "Resistor_SMD:R_0402_1005Metric"
 			(at 77.47 53.34 0)
 			(hide yes)
@@
 			)
 		)
-		(property "Footprint" "Capacitor_SMD:C_0603_1608Metric"
+		(property "Footprint" "Capacitor_SMD:C_0402_1005Metric"
 			(at 43.18 254.3048 0)
 			(hide yes)
@@
 			)
 		)
-		(property "Footprint" "Capacitor_SMD:C_0603_1608Metric"
+		(property "Footprint" "Capacitor_SMD:C_0402_1005Metric"
 			(at 31.75 52.07 0)
 			(hide yes)
@@
 			)
 		)
-		(property "Footprint" "Resistor_SMD:R_0603_1608Metric"
+		(property "Footprint" "Resistor_SMD:R_0402_1005Metric"
 			(at 77.47 63.5 0)
 			(hide yes)

Commit message: more rev2 changes
Parts:
- removed C29: 1u, Capacitor_SMD:C_0603_1608Metric, symbol Device:C
- removed R17: 100k, Resistor_SMD:R_0402_1005Metric, symbol Device:R
- removed R18: 200k, Resistor_SMD:R_0402_1005Metric, symbol Device:R
- removed R27, R29, R30: 0, Jumper:SolderJumper-2_P1.3mm_Bridged_RoundedPad1.0x1.5mm, symbol Device:R_Small
- removed TP1: TestPoint, TestPoint:TestPoint_Pad_D1.5mm, symbol Connector:TestPoint
- added C72: 1n, Capacitor_SMD:C_0402_1005Metric, symbol Device:C_Small
- added J12: PYRO_2_B, Connector_Molex:Molex_Nano-Fit_105313-xx02_1x02_P2.50mm_Horizontal, symbol Connector_Generic:Conn_01x02
- added J13: PYRO_1_B, Connector_Molex:Molex_Nano-Fit_105313-xx02_1x02_P2.50mm_Horizontal, symbol Connector_Generic:Conn_01x02
- added R42: 200k, Resistor_SMD:R_0402_1005Metric, symbol Device:R_Small
- added R43: 39k, Resistor_SMD:R_0402_1005Metric, symbol Device:R_Small
- R26, R34: value 100k -> 39k
Connections:
- net BAT: now also J12.2 (Pin_2), J13.2 (Pin_2), R42.1
- net GND: now also C72.2, R43.2
- net GPIO26_ADC0: now also U4.40 (GPIO26_ADC0), C72.1, R42.2, R43.1
- net GPIO28_ADC2: now also U4.42 (GPIO28_ADC2)
- net GPIO29_ADC3: now also U4.43 (GPIO29_ADC3)
- net at J6.2 (Pin_2), Q5.3 (D), R24.2: now also J13.1 (Pin_1)
- net at J10.2 (Pin_2), Q6.3 (D), R32.2: now also J12.1 (Pin_1)
Other:
- moved on the sheet: C26, C28, C58, C59, C60, C61, C62, C64, C7, D2, J4, L14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

Commit message: extra connector
Parts:
- added J2: Extra Connection, Connector_Molex:Molex_PicoBlade_53047-0410_1x04_P1.25mm_Vertical, symbol Connector_Generic:Conn_01x04
- added TP1: SWCLK, TestPoint:TestPoint_Pad_D1.5mm, symbol Connector:TestPoint
- added TP4: SWD, TestPoint:TestPoint_Pad_D1.5mm, symbol Connector:TestPoint
Connections:
- net +3V3: now also J2.3 (Pin_3)
- net +5V: now also J2.4 (Pin_4)
- net GND: now also J2.1 (Pin_1)
- net SWCLK: now also TP1.1
- net SWD: now also TP4.1
- net GPIO27_ADC1: now reaches U4.41 (GPIO27_ADC1)
- net GPIO27_ADC1: now also J2.2 (Pin_2)
- no-connect marks 7 -> 6
Other:
- note added: "Misc connectors"
